Commit message: commented and cleaned up code, add derivative control to v controller

File: quad_model/urdf/map.urdf (robot description, URDF)
Before this commit: robot ${robot_name}, 1 links, 0 joints
Links:
- link map: geometry collision mesh filename=package://quad_model/meshes/scan3.obj scale=3 3 3; visual mesh filename=package://quad_model/meshes/scan3.obj scale=3 3 3

Commit message: updated sim to get rid of negative motor force and handle high frequency update rates from sim node, decoupled the convergence time from update rate for smoother trajectories

File: quad_model/urdf/map.urdf (robot description, URDF)
Before this commit: robot ${robot_name}, 1 links, 0 joints
Links:
- link map: geometry collision mesh filename=package://quad_model/meshes/scan3.obj scale=4 4 4; visual mesh filename=package://quad_model/meshes/scan3.obj scale=4 4 4

Commit message: Incredibly efficient A* with KDTree, also new map and integral control

File: quad_model/urdf/map.urdf (robot description, URDF)
Before this commit: robot ${robot_name}, 1 links, 0 joints
Links:
- link map: geometry collision mesh filename=package://quad_model/meshes/city.obj scale=1 1 1; visual mesh filename=package://quad_model/meshes/city.obj scale=1 1 1
